Commit message: Finalize the gazebo environments

File: ur3_description/urdf/realsense_rs435.urdf.xacro (robot description, xacro)
@@ -4,67 +4,74 @@
     <xacro:arg name="add_plug" default="true"/>
     <xacro:include filename="$(find realsense2_description)/urdf/_d435.urdf.xacro" />
-    <link name="world" />
-    <link name="global_camera">
-        <inertial>
-        <origin rpy="0 0 0" xyz="0 0 0"/>
-        <mass value="0.0001"/>
-        <inertia ixx="1e-08" ixy="0" ixz="0" iyy="1e-08" iyz="0" izz="1e-08"/>
-        </inertial>
-    </link>
-    <xacro:sensor_d435 parent="global_camera" use_nominal_extrinsics="$(arg use_nominal_extrinsics)">
-        <origin xyz="0 0 0" rpy="0 0 0"/>
-    </xacro:sensor_d435>
-    <joint name="global_camera" type="fixed">
-        <origin rpy="0 0 0" xyz="0 0 0"/>
-        <parent link="world"/>
-        <child link="global_camera"/>
-    </joint>
-    <!-- camera -->
-    <gazebo reference="global_camera">
-        <sensor name="global_camera" type="depth">
-            <update_rate>20</update_rate>
-            <camera name="global_camera">
-                <horizontal_fov>1.047</horizontal_fov>
-                <image>
-                    <width>640</width>
-                    <height>480</height>
-                    <format>RGB_INT8</format>
-                </image>
-                <clip>
-                    <near>0.1</near>
-                    <far>100</far>
-                </clip>
-                <noise>
-                    <type>gaussian</type>
-                    <mean>0.0</mean>
-                    <stddev>0.007</stddev>
-                </noise>
-                <visualize>1</visualize>
-            </camera>
-            <plugin name="camera_controller" filename="libgazebo_ros_openni_kinect.so">
-                <baseline>0.2</baseline>
-                <alwaysOn>true</alwaysOn>
-                <updateRate>60.0</updateRate>
-                <cameraName>global_camera</cameraName>
-                <imageTopicName>/camera/color/image_raw</imageTopicName>
-                <cameraInfoTopicName>/camera/color/camera_info</cameraInfoTopicName>
-                <depthImageTopicName>/camera/depth/image_raw</depthImageTopicName>
-                <depthImageInfoTopicName>/camera/depth/camera_info</depthImageInfoTopicName>
-                <pointCloudTopicName>/camera/depth/points</pointCloudTopicName>
-                <frameName>global_camera</frameName>
-                <pointCloudCutoff>0.5</pointCloudCutoff>
-                <pointCloudCutoffMax>3.0</pointCloudCutoffMax>
-                <distortionK1>0.00000001</distortionK1>
-                <distortionK2>0.00000001</distortionK2>
-                <distortionK3>0.00000001</distortionK3>
-                <distortionT1>0.00000001</distortionT1>
-                <distortionT2>0.00000001</distortionT2>
-                <CxPrime>0</CxPrime>
-                <Cx>0</Cx>
-                <Cy>0</Cy>
-                <focalLength>0</focalLength>
-                <hackBaseline>0</hackBaseline>
-            </plugin>
-        </sensor>
-    </gazebo>
+    <xacro:macro name="realsense2_camera" params="prefix parent *origin">
+        <link name="global_camera">
+            <inertial>
+            <origin rpy="0 0 0" xyz="0 0 0"/>
+            <mass value="0.0001"/>
+            <inertia ixx="1e-08" ixy="0" ixz="0" iyy="1e-08" iyz="0" izz="1e-08"/>
+            </inertial>
+        </link>
+        <xacro:sensor_d435 parent="global_camera" use_nominal_extrinsics="$(arg use_nominal_extrinsics)">
+            <origin xyz="0 0 0" rpy="0 0 0"/>
+        </xacro:sensor_d435>
+        <joint name="${prefix}global_camera" type="fixed">
+            <parent link="${parent}"/>
+            <child link="global_camera"/>
+            <xacro:insert_block name="origin"/>
+        </joint>
+        <!-- <joint name="camera_depth_joint" type="fixed">
+            <origin xyz="0 0 0" rpy="${-pi/2} 0 ${-pi/2} "/>
+            <parent link="camera_link"/>
+            <child link="camera_depth_link"/>
+        </joint>
+        <link name="camera_depth_link"/> -->
+        <!-- camera -->
+        <gazebo reference="global_camera">
+            <sensor name="global_camera" type="depth">
+                <update_rate>20</update_rate>
+                <camera name="global_camera">
+                    <horizontal_fov>1.047</horizontal_fov>
+                    <image>
+                        <width>640</width>
+                        <height>480</height>
+                        <format>RGB_INT8</format>
+                    </image>
+                    <clip>
+                        <near>0.1</near>
+                        <far>100</far>
+                    </clip>
+                    <noise>
+                        <type>gaussian</type>
+                        <mean>0.0</mean>
+                        <stddev>0.007</stddev>
+                    </noise>
+                    <visualize>1</visualize>
+                </camera>
+                <plugin name="camera_controller" filename="libgazebo_ros_openni_kinect.so">
+                    <baseline>0.2</baseline>
+                    <alwaysOn>true</alwaysOn>
+                    <updateRate>60.0</updateRate>
+                    <cameraName>global_camera</cameraName>
+                    <imageTopicName>/camera/color/image_raw</imageTopicName>
+                    <cameraInfoTopicName>/camera/color/camera_info</cameraInfoTopicName>
+                    <depthImageTopicName>/camera/depth/image_raw</depthImageTopicName>
+                    <depthImageInfoTopicName>/camera/depth/camera_info</depthImageInfoTopicName>
+                    <pointCloudTopicName>/camera/depth/points</pointCloudTopicName>
+                    <frameName>camera_depth_optical_frame</frameName>
+                    <pointCloudCutoff>0.1</pointCloudCutoff>
+                    <pointCloudCutoffMax>3.0</pointCloudCutoffMax>
+                    <distortionK1>0.00000001</distortionK1>
+                    <distortionK2>0.00000001</distortionK2>
+                    <distortionK3>0.00000001</distortionK3>
+                    <distortionT1>0.00000001</distortionT1>
+                    <distortionT2>0.00000001</distortionT2>
+                    <CxPrime>0</CxPrime>
+                    <Cx>0</Cx>
+                    <Cy>0</Cy>
+                    <focalLength>0</focalLength>
+                    <hackBaseline>0</hackBaseline>
+                </plugin>
+            </sensor>
+        </gazebo>
+  </xacro:macro>
 </robot>

Commit message: Update heuristics grasp attach

File: ur3_description/urdf/realsense_rs435.urdf.xacro (robot description, xacro)
@@ -2,33 +2,15 @@
 <robot name="realsense2_camera" xmlns:xacro="http://ros.org/wiki/xacro">
     <xacro:arg name="use_nominal_extrinsics" default="true"/>
-    <xacro:arg name="add_plug" default="true"/>
+    <xacro:arg name="add_plug" default="false" />
+    <xacro:arg name="use_mesh" default="true" />
     <xacro:include filename="$(find realsense2_description)/urdf/_d435.urdf.xacro" />
     <xacro:macro name="realsense2_camera" params="prefix parent *origin">
-        <link name="global_camera">
-            <inertial>
-            <origin rpy="0 0 0" xyz="0 0 0"/>
-            <mass value="0.0001"/>
-            <inertia ixx="1e-08" ixy="0" ixz="0" iyy="1e-08" iyz="0" izz="1e-08"/>
-            </inertial>
-        </link>
-        <xacro:sensor_d435 parent="global_camera" use_nominal_extrinsics="$(arg use_nominal_extrinsics)">
-            <origin xyz="0 0 0" rpy="0 0 0"/>
+        <xacro:sensor_d435 parent="${parent}" use_nominal_extrinsics="$(arg use_nominal_extrinsics)" add_plug="$(arg add_plug)" use_mesh="$(arg use_mesh)">
+            <xacro:insert_block name="origin"/>
         </xacro:sensor_d435>
-        <joint name="${prefix}global_camera" type="fixed">
-            <parent link="${parent}"/>
-            <child link="global_camera"/>
-            <xacro:insert_block name="origin"/>
-        </joint>
-        <!-- <joint name="camera_depth_joint" type="fixed">
-            <origin xyz="0 0 0" rpy="${-pi/2} 0 ${-pi/2} "/>
-            <parent link="camera_link"/>
-            <child link="camera_depth_link"/>
-        </joint>
-        <link name="camera_depth_link"/> -->
-        <!-- camera -->
-        <gazebo reference="global_camera">
-            <sensor name="global_camera" type="depth">
+        <gazebo reference="camera_link">
+            <sensor name="camera" type="depth">
                 <update_rate>20</update_rate>
-                <camera name="global_camera">
+                <camera name="camera">
                     <horizontal_fov>1.047</horizontal_fov>
                     <image>
@@ -51,5 +33,5 @@
                     <baseline>0.2</baseline>
                     <alwaysOn>true</alwaysOn>
-                    <updateRate>60.0</updateRate>
+                    <updateRate>10</updateRate>
                     <cameraName>global_camera</cameraName>
                     <imageTopicName>/camera/color/image_raw</imageTopicName>
@@ -74,4 +56,4 @@
             </sensor>
         </gazebo>
-  </xacro:macro>
+    </xacro:macro>
 </robot>

File: ur3_gazebo/urdf/ur_gripper_85_realsense.xacro (robot description, xacro)
@@ -116,5 +116,5 @@
   <!-- Attach realsense -->
   <xacro:realsense2_camera prefix="" parent="robotiq_coupler" >
-    <origin xyz="0.1 0 0" rpy="0 ${-pi/2} ${pi}"/>
+    <origin xyz="0.08 0 0" rpy="0 ${-pi/2} ${pi}"/>
   </xacro:realsense2_camera>
   <!-- Gazebo Force/Torque sensor plugin -->
@@ -137,9 +137,39 @@
       grasp_plugin True = custom gazebo_grasp_fix
   -->
-  <xacro:if value="$(arg grasp_plugin)">
+  <gazebo reference="robotiq_85_left_finger_tip_link">
+    <sensor name="main_bumper" type="contact">
+        <selfCollide>true</selfCollide>
+        <alwaysOn>true</alwaysOn>
+        <updateRate>50.0</updateRate>
+        <material>Gazebo/Red</material>
+        <contact>
+          <collision>robotiq_85_left_finger_tip_link_collision</collision>
+        </contact>
+        <plugin name="gazebo_ros_bumper_controller" filename="libgazebo_ros_bumper.so">
+          <bumperTopicName>robotiq_85_left_finger_tip_link_contacts</bumperTopicName>
+          <frameName>robotiq_85_left_finger_tip_link</frameName>
+        </plugin>
+    </sensor>
+  </gazebo>
+  <gazebo reference="robotiq_85_right_finger_tip_link">
+    <sensor name="main_bumper" type="contact">
+        <selfCollide>true</selfCollide>
+        <alwaysOn>true</alwaysOn>
+        <updateRate>50.0</updateRate>
+        <material>Gazebo/Red</material>
+        <contact>
+          <collision>robotiq_85_right_finger_tip_link_collision</collision>
+        </contact>
+        <plugin name="gazebo_ros_bumper_controller" filename="libgazebo_ros_bumper.so">
+          <bumperTopicName>robotiq_85_right_finger_tip_link_contacts</bumperTopicName>
+          <frameName>robotiq_85_right_finger_tip_link</frameName>
+        </plugin>
+    </sensor>
+  </gazebo>
+  <!-- <xacro:if value="$(arg grasp_plugin)">
     <gazebo>
       <plugin name="gazebo_grasp_fix" filename="libgazebo_grasp_fix.so">
             <arm>
-              <arm_name>robotiq_85</arm_name>
+              <arm_name>robot</arm_name>
               <palm_link>wrist_3_link</palm_link>
               <gripper_link>robotiq_85_left_finger_tip_link</gripper_link>
@@ -147,8 +177,8 @@
             </arm>
           <forces_angle_tolerance>100</forces_angle_tolerance>
-          <update_rate>100</update_rate>
-          <grip_count_threshold>5</grip_count_threshold>
-          <max_grip_count>30</max_grip_count>
-          <release_tolerance>0.0015</release_tolerance>
+          <update_rate>5</update_rate>
+          <grip_count_threshold>3</grip_count_threshold>
+          <max_grip_count>8</max_grip_count>
+          <release_tolerance>0.005</release_tolerance>
           <disable_collisions_on_attach>false</disable_collisions_on_attach>
           <contact_topic>__default_topic__</contact_topic>
@@ -169,5 +199,5 @@
       </gripper>
     </gazebo>
-  </xacro:unless>
+  </xacro:unless> -->
   <!-- Gazebo grasping plugin -->
 </robot>
